File: kicad/modubu.kicad_pcb (KiCad board)
At the start: 2 copper layers, 100 x 92 mm, 45 parts, among them J1 AudioJack4, J2 AudioJack4, SW1 SW_Push, SW10 SW_Push, SW11 SW_Push, SW12 SW_Push, SW13 SW_Push, SW14 SW_Push, SW15 SW_Push, SW16 SW_Push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

Commit message: add board art
Parts:
- added G***: LOGO, modubu-CustomFoot:meshgradation, F.Cu at (90.5, 100.5)
- added G***: LOGO, modubu-CustomFoot:meshgradation, B.Cu at (90.5, 100.5)
