File: kicad/modubuSolder.kicad_pcb (KiCad board)
At the start: 2 copper layers, 100 x 92 mm, 47 parts, among them J1 AudioJack4, J2 AudioJack4, SW1 SW_Push, SW10 SW_Push, SW11 SW_Push, SW12 SW_Push, SW13 SW_Push, SW14 SW_Push, SW15 SW_Push, SW16 SW_Push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

Commit message: polish up board art
Parts:
- G***: footprint modubu-CustomFoot:meshgradation -> modubu-CustomFoot:meshgradationNameHole1
- G***: footprint modubu-CustomFoot:meshgradation -> modubu-CustomFoot:meshgradationNameHole2
